File: ProjecteRobotPAE.kicad_sch (KiCad schematic)
At the start: 0 parts

Commit message: Afegir micro
Parts:
- added U1: PIC16LF18446-I_P, PIC16LF18446-I_P:DIP793W45P254L2590H533Q20, symbol MCU_Microchip_PIC16:PIC16LF18446-I_P
Connections:
- new net GND: U1.20 (VSS)

Commit message: 2/7/2025 sensors i micro
Parts:
- removed U1: PIC16LF18446-I_P, PIC16LF18446-I_P:DIP793W45P254L2590H533Q20, symbol MCU_Microchip_PIC16:PIC16LF18446-I_P
- added C1: C, symbol Device:C
- added J3: Conn_01x05_Pin, Connector_PinHeader_2.54mm:PinHeader_1x05_P2.54mm_Vertical, symbol Connector:Conn_01x05_Pin
- added U1: PIC16F18426-I/ST, TSSOP14_ST_MCH, symbol 2025-07-02_10-07-00:PIC16F18426-I_ST
- added U2, U3, U4: AM2302, Sensor:ASAIR_AM2302_P2.54mm_Vertical, symbol Sensor:AM2302
Connections:
- net GND: now also J3.3 (Pin_3), U1.14 (VSS), U2.2 (GND), U3.2 (GND), U4.2 (GND)
- new net: C1.1, U1.1 (VDD)
- new net MCLR: J3.1 (Pin_1), U1.4 (MCLR/VPP/RA3)
- new net PGC: J3.5 (Pin_5), U1.12 (RA1/ICSPCLK)
- new net PGD: J3.4 (Pin_4), U1.13 (RA0/ICSPDAT)
- new net RX/TX: U1.5 (RC5), U1.6 (RC4)
- new net S1: U1.10 (RC0), U2.1 (V0)
- new net S2: U1.9 (RC1), U3.1 (V0)
- new net S3: U1.8 (RC2), U4.1 (V0)
- new net VCC: U2.3 (VCC), U2.4 (GND), U3.3 (VCC), U3.4 (GND), U4.3 (VCC), U4.4 (GND)
- new net Vcc: J3.2 (Pin_2)
Other:
- note added: "ICSP"
- note added: "Sensors"
